File: kicad/shield/pcb.kicad_pcb (KiCad board)
At the start: 2 copper layers, 48.9 x 49.5 mm, 14 parts, among them J1 Conn_01x12_Fem_l, J2 Conn_01x12_Fem_r, J3 Conn_01x12_Fem_b_r, J4 Conn_01x09_Fem_b_l

Commit message: maybe final
- ultimate PCB design
- add potentiometer for led control
- checked connections
Parts:
- added R2: 2 kOhm, Potentiometers:Potentiometer_Triwood_RM-065, F.Cu at (93.5, 100.6)
- R1: value 82 Ohm -> 100 Ohm
- moved C3 20.2 mm to (124.5, 97.0)
- moved C1 11.7 mm to (117.9, 106.2)
- moved R1 10.7 mm to (107.2, 97.0), turned to 270 degrees
- moved J4 3.30 mm to (92.5, 71.1)
- moved D1 1.63 mm to (100.1, 106.7)
- moved C2 0.40 mm to (117.9, 99.6)
Connections:
- net 12 renamed 21
- R1 pad 2: Net-(D1-Pad2) -> Net-(R1-Pad2)
Routing:
- net A0: track 0.00 -> 53.0 mm
- net A2: track 0.00 -> 44.8 mm
- net A1: track 0.00 -> 44.4 mm, vias 0 -> 1
- net Net-(D1-Pad2): track 0.00 -> 43.6 mm
- net Net-(R1-Pad2): track 0.00 -> 22.1 mm
- net 1: track 0.00 -> 18.2 mm
- net 8: track 0.00 -> 17.1 mm
- net 6: track 0.00 -> 17.1 mm
- net 5: track 0.00 -> 17.1 mm
- net 3: track 0.00 -> 17.1 mm
- net 0: track 0.00 -> 17.1 mm
- net 9: track 0.00 -> 17.1 mm
- net 7: track 0.00 -> 17.1 mm
- net 4: track 0.00 -> 17.1 mm
- net 2: track 0.00 -> 17.1 mm
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- added copper zone on B.Cu, net GND
