File: kicad/shield_touch/_saved_pcb.sch (KiCad schematic (older format))
At the start: 22 parts, among them J1 Conn_01x12_Fem_l, J2 Conn_01x12_Fem_r, J3 Conn_01x09_Fem_b_l

Commit message: update
- still to fix
Parts:
- gave numbers to parts that had none: 1
Changed lines of the file:
@@
 $EndComp
 $Comp
-L GND #PWR01
+L GND #PWR1
 U 1 1 5A7C61AA
 P 1560 4990
-F 0 "#PWR01" H 1560 4740 50  0001 C CNN
+F 0 "#PWR1" H 1560 4740 50  0001 C CNN
 F 1 "GND" H 1560 4840 50  0000 C CNN
 F 2 "" H 1560 4990 50  0001 C CNN
@@
 21
 $Comp
-L GND #PWR02
+L GND #PWR3
 U 1 1 5A7C7797
 P 6290 5320
-F 0 "#PWR02" H 6290 5070 50  0001 C CNN
+F 0 "#PWR3" H 6290 5070 50  0001 C CNN
 F 1 "GND" H 6290 5170 50  0000 C CNN
 F 2 "" H 6290 5320 50  0001 C CNN
@@
 A2
 $Comp
-L GND #PWR03
+L GND #PWR2
 U 1 1 5A7C90CD
 P 5530 3110
-F 0 "#PWR03" H 5530 2860 50  0001 C CNN
+F 0 "#PWR2" H 5530 2860 50  0001 C CNN
 F 1 "GND" H 5530 2960 50  0000 C CNN
 F 2 "" H 5530 3110 50  0001 C CNN
@@
 1
 $Comp
-L GND #PWR04
+L GND #PWR4
 U 1 1 5A7CA9FF
 P 7020 5320
-F 0 "#PWR04" H 7020 5070 50  0001 C CNN
+F 0 "#PWR4" H 7020 5070 50  0001 C CNN
 F 1 "GND" H 7020 5170 50  0000 C CNN
 F 2 "" H 7020 5320 50  0001 C CNN
@@
 Connection ~ 1560 4320
 Wire Wire Line
-	1560 2430 1560 4050
-Wire Wire Line
-	1560 4050 1560 4320
-Wire Wire Line
-	1560 4320 1560 4620
-Wire Wire Line
-	1560 4620 1560 4990
+	1560 2430 1560 4990
 Wire Wire Line
 	1760 4620 1560 4620
@@
 	2320 4050 2320 1830
 Wire Wire Line
-	2220 1830 2320 1830
-Wire Wire Line
-	2320 1830 3100 1830
+	2220 1830 3100 1830
 Wire Wire Line
 	2460 4320 2460 1930
 Wire Wire Line
-	2220 1930 2460 1930
-Wire Wire Line
-	2460 1930 3100 1930
+	2220 1930 3100 1930
 Wire Wire Line
 	6170 5050 6290 5050
@@
 	2610 4620 2610 2030
 Wire Wire Line
-	2220 2030 2610 2030
-Wire Wire Line
-	2610 2030 3100 2030
+	2220 2030 3100 2030
 Connection ~ 2610 2030
 Wire Wire Line
 	5060 2240 5530 2240
 Wire Wire Line
-	5530 2240 5530 2340
-Wire Wire Line
-	5530 2340 5530 3110
+	5530 2240 5530 3110
 Wire Wire Line
 	5060 2340 5530 2340
@@
 VCC
 Wire Wire Line
-	4010 3580 4190 3580
-Wire Wire Line
-	4190 3580 4620 3580
+	4010 3580 4620 3580
 Wire Wire Line
 	4010 3780 4190 3780
 Wire Wire Line
-	4190 3580 4190 3780
-Wire Wire Line
-	4190 3780 4190 3980
-Wire Wire Line
-	4190 3980 4190 4180
-Wire Wire Line
-	4190 4180 4190 4370
-Wire Wire Line
-	4190 4370 4190 4570
-Wire Wire Line
-	4190 4570 4190 4770
-Wire Wire Line
-	4190 4770 4190 4970
-Wire Wire Line
-	4190 4970 4190 5150
-Wire Wire Line
-	4190 5150 4190 5350
-Wire Wire Line
-	4190 5350 4190 5550
-Wire Wire Line
-	4190 5550 4190 5750
-Wire Wire Line
-	4190 5750 4190 5940
-Wire Wire Line
-	4190 5940 4190 6140
-Wire Wire Line
-	4190 6140 4190 6340
+	4190 3580 4190 6340
 Connection ~ 4190 3580
 Wire Wire Line
@@
 	3560 6340 3710 6340
 $Comp
-L Conn_01x11_Fem_b_r_touch J?
+L Conn_01x11_Fem_b_r_touch J4
 U 1 1 5B002141
 P 7560 4600
-F 0 "J?" H 7560 5200 50  0000 C CNN
+F 0 "J4" H 7560 5200 50  0000 C CNN
 F 1 "Conn_01x11_Fem_b_r_touch" H 8070 3960 50  0000 C CNN
 F 2 "Connectors_Samtec:SL-111-X-XX_1x11" H 7560 4600 50  0001 C CNN
