File: kicad/shield_touch/pcb.sch (KiCad schematic (older format))
At the start: 22 parts, among them J1 Conn_01x12_Fem_l, J2 Conn_01x12_Fem_r, J3 Conn_01x09_Fem_b_l, J4 Conn_01x11_Fem_b_r_touch

Commit message: update
- designing pcb with vertical resistors
Parts:
- R1, R10, R11, R12, R13, R14, R15, R2, R3, R4, R5, R6, R7, R8, R9: footprint Resistors_THT:R_Axial_DIN0207_L6.3mm_D2.5mm_P10.16mm_Horizontal -> Resistors_THT:R_Axial_DIN0204_L3.6mm_D1.6mm_P2.54mm_Vertical
Changed lines of the file:
@@
 $EndComp
 $Comp
-L GND #PWR1
+L GND #PWR01
 U 1 1 5A7C61AA
 P 1560 4990
-F 0 "#PWR1" H 1560 4740 50  0001 C CNN
+F 0 "#PWR01" H 1560 4740 50  0001 C CNN
 F 1 "GND" H 1560 4840 50  0000 C CNN
 F 2 "" H 1560 4990 50  0001 C CNN
@@
 21
 $Comp
-L GND #PWR3
+L GND #PWR02
 U 1 1 5A7C7797
 P 6290 5320
-F 0 "#PWR3" H 6290 5070 50  0001 C CNN
+F 0 "#PWR02" H 6290 5070 50  0001 C CNN
 F 1 "GND" H 6290 5170 50  0000 C CNN
 F 2 "" H 6290 5320 50  0001 C CNN
@@
 A2
 $Comp
-L GND #PWR2
+L GND #PWR03
 U 1 1 5A7C90CD
 P 5530 3110
-F 0 "#PWR2" H 5530 2860 50  0001 C CNN
+F 0 "#PWR03" H 5530 2860 50  0001 C CNN
 F 1 "GND" H 5530 2960 50  0000 C CNN
 F 2 "" H 5530 3110 50  0001 C CNN
@@
 1
 $Comp
-L GND #PWR4
+L GND #PWR04
 U 1 1 5A7CA9FF
 P 7020 5320
-F 0 "#PWR4" H 7020 5070 50  0001 C CNN
+F 0 "#PWR04" H 7020 5070 50  0001 C CNN
 F 1 "GND" H 7020 5170 50  0000 C CNN
 F 2 "" H 7020 5320 50  0001 C CNN
@@
 F 0 "R1" V 3940 3580 50  0000 C CNN
 F 1 "2M" V 3860 3580 50  0000 C CNN
-F 2 "Resistors_THT:R_Axial_DIN0207_L6.3mm_D2.5mm_P10.16mm_Horizontal" V 3790 3580 50  0001 C CNN
+F 2 "Resistors_THT:R_Axial_DIN0204_L3.6mm_D1.6mm_P2.54mm_Vertical" V 3790 3580 50  0001 C CNN
 F 3 "" H 3860 3580 50  0001 C CNN
 	1    3860 3580
@@
 F 0 "R2" V 3940 3780 50  0000 C CNN
 F 1 "2M" V 3860 3780 50  0000 C CNN
-F 2 "Resistors_THT:R_Axial_DIN0207_L6.3mm_D2.5mm_P10.16mm_Horizontal" V 3790 3780 50  0001 C CNN
+F 2 "Resistors_THT:R_Axial_DIN0204_L3.6mm_D1.6mm_P2.54mm_Vertical" V 3790 3780 50  0001 C CNN
 F 3 "" H 3860 3780 50  0001 C CNN
 	1    3860 3780
@@
 F 0 "R3" V 3940 3980 50  0000 C CNN
 F 1 "2M" V 3860 3980 50  0000 C CNN
-F 2 "Resistors_THT:R_Axial_DIN0207_L6.3mm_D2.5mm_P10.16mm_Horizontal" V 3790 3980 50  0001 C CNN
+F 2 "Resistors_THT:R_Axial_DIN0204_L3.6mm_D1.6mm_P2.54mm_Vertical" V 3790 3980 50  0001 C CNN
 F 3 "" H 3860 3980 50  0001 C CNN
 	1    3860 3980
@@
 F 0 "R4" V 3940 4180 50  0000 C CNN
 F 1 "2M" V 3860 4180 50  0000 C CNN
-F 2 "Resistors_THT:R_Axial_DIN0207_L6.3mm_D2.5mm_P10.16mm_Horizontal" V 3790 4180 50  0001 C CNN
+F 2 "Resistors_THT:R_Axial_DIN0204_L3.6mm_D1.6mm_P2.54mm_Vertical" V 3790 4180 50  0001 C CNN
 F 3 "" H 3860 4180 50  0001 C CNN
 	1    3860 4180
@@
 F 0 "R5" V 3940 4370 50  0000 C CNN
 F 1 "2M" V 3860 4370 50  0000 C CNN
-F 2 "Resistors_THT:R_Axial_DIN0207_L6.3mm_D2.5mm_P10.16mm_Horizontal" V 3790 4370 50  0001 C CNN
+F 2 "Resistors_THT:R_Axial_DIN0204_L3.6mm_D1.6mm_P2.54mm_Vertical" V 3790 4370 50  0001 C CNN
 F 3 "" H 3860 4370 50  0001 C CNN
 	1    3860 4370
@@
 F 0 "R6" V 3940 4570 50  0000 C CNN
 F 1 "2M" V 3860 4570 50  0000 C CNN
-F 2 "Resistors_THT:R_Axial_DIN0207_L6.3mm_D2.5mm_P10.16mm_Horizontal" V 3790 4570 50  0001 C CNN
+F 2 "Resistors_THT:R_Axial_DIN0204_L3.6mm_D1.6mm_P2.54mm_Vertical" V 3790 4570 50  0001 C CNN
 F 3 "" H 3860 4570 50  0001 C CNN
 	1    3860 4570
@@
 F 0 "R7" V 3940 4770 50  0000 C CNN
 F 1 "2M" V 3860 4770 50  0000 C CNN
-F 2 "Resistors_THT:R_Axial_DIN0207_L6.3mm_D2.5mm_P10.16mm_Horizontal" V 3790 4770 50  0001 C CNN
+F 2 "Resistors_THT:R_Axial_DIN0204_L3.6mm_D1.6mm_P2.54mm_Vertical" V 3790 4770 50  0001 C CNN
 F 3 "" H 3860 4770 50  0001 C CNN
 	1    3860 4770
@@
 F 0 "R8" V 3940 4970 50  0000 C CNN
 F 1 "2M" V 3860 4970 50  0000 C CNN
-F 2 "Resistors_THT:R_Axial_DIN0207_L6.3mm_D2.5mm_P10.16mm_Horizontal" V 3790 4970 50  0001 C CNN
+F 2 "Resistors_THT:R_Axial_DIN0204_L3.6mm_D1.6mm_P2.54mm_Vertical" V 3790 4970 50  0001 C CNN
 F 3 "" H 3860 4970 50  0001 C CNN
 	1    3860 4970
@@
 F 0 "R9" V 3940 5150 50  0000 C CNN
 F 1 "2M" V 3860 5150 50  0000 C CNN
-F 2 "Resistors_THT:R_Axial_DIN0207_L6.3mm_D2.5mm_P10.16mm_Horizontal" V 3790 5150 50  0001 C CNN
+F 2 "Resistors_THT:R_Axial_DIN0204_L3.6mm_D1.6mm_P2.54mm_Vertical" V 3790 5150 50  0001 C CNN
 F 3 "" H 3860 5150 50  0001 C CNN
 	1    3860 5150
@@
 F 0 "R10" V 3940 5350 50  0000 C CNN
 F 1 "2M" V 3860 5350 50  0000 C CNN
-F 2 "Resistors_THT:R_Axial_DIN0207_L6.3mm_D2.5mm_P10.16mm_Horizontal" V 3790 5350 50  0001 C CNN
+F 2 "Resistors_THT:R_Axial_DIN0204_L3.6mm_D1.6mm_P2.54mm_Vertical" V 3790 5350 50  0001 C CNN
 F 3 "" H 3860 5350 50  0001 C CNN
 	1    3860 5350
@@
 F 0 "R11" V 3940 5550 50  0000 C CNN
 F 1 "2M" V 3860 5550 50  0000 C CNN
-F 2 "Resistors_THT:R_Axial_DIN0207_L6.3mm_D2.5mm_P10.16mm_Horizontal" V 3790 5550 50  0001 C CNN
+F 2 "Resistors_THT:R_Axial_DIN0204_L3.6mm_D1.6mm_P2.54mm_Vertical" V 3790 5550 50  0001 C CNN
 F 3 "" H 3860 5550 50  0001 C CNN
 	1    3860 5550
@@
 F 0 "R12" V 3940 5750 50  0000 C CNN
 F 1 "2M" V 3860 5750 50  0000 C CNN
-F 2 "Resistors_THT:R_Axial_DIN0207_L6.3mm_D2.5mm_P10.16mm_Horizontal" V 3790 5750 50  0001 C CNN
+F 2 "Resistors_THT:R_Axial_DIN0204_L3.6mm_D1.6mm_P2.54mm_Vertical" V 3790 5750 50  0001 C CNN
 F 3 "" H 3860 5750 50  0001 C CNN
 	1    3860 5750
@@
 F 0 "R13" V 3940 5940 50  0000 C CNN
 F 1 "2M" V 3860 5940 50  0000 C CNN
-F 2 "Resistors_THT:R_Axial_DIN0207_L6.3mm_D2.5mm_P10.16mm_Horizontal" V 3790 5940 50  0001 C CNN
+F 2 "Resistors_THT:R_Axial_DIN0204_L3.6mm_D1.6mm_P2.54mm_Vertical" V 3790 5940 50  0001 C CNN
 F 3 "" H 3860 5940 50  0001 C CNN
 	1    3860 5940
@@
 F 0 "R14" V 3940 6140 50  0000 C CNN
 F 1 "2M" V 3860 6140 50  0000 C CNN
-F 2 "Resistors_THT:R_Axial_DIN0207_L6.3mm_D2.5mm_P10.16mm_Horizontal" V 3790 6140 50  0001 C CNN
+F 2 "Resistors_THT:R_Axial_DIN0204_L3.6mm_D1.6mm_P2.54mm_Vertical" V 3790 6140 50  0001 C CNN
 F 3 "" H 3860 6140 50  0001 C CNN
 	1    3860 6140
@@
 F 0 "R15" V 3940 6340 50  0000 C CNN
 F 1 "2M" V 3860 6340 50  0000 C CNN
-F 2 "Resistors_THT:R_Axial_DIN0207_L6.3mm_D2.5mm_P10.16mm_Horizontal" V 3790 6340 50  0001 C CNN
+F 2 "Resistors_THT:R_Axial_DIN0204_L3.6mm_D1.6mm_P2.54mm_Vertical" V 3790 6340 50  0001 C CNN
 F 3 "" H 3860 6340 50  0001 C CNN
 	1    3860 6340
