File: kicad/touch_buttons/touch.sch (KiCad schematic (older format))
At the start: 31 parts

Commit message: update
Parts:
- removed J?: CONN_01X17, symbol CONN_01X17
- removed JP10, JP11, JP12, JP13, JP14, JP2, JP3, JP4, JP5, JP6, JP7, JP8, JP9, JP?: touch, symbol Jumper_NO_Small
- removed R? (x15): R, symbol R
- added 2M: R, symbol R
- added J1: CONN_01X03, symbol CONN_01X03
Connections:
- net GND: now also JP1.1, J1.3 (P3)
- net at JP1.2: now also 2M.2, J1.2 (P2)
- new net: 2M.1, J1.1 (P1)
Other:
- note added: "Finger"
- note added: "GND"
- note added: "IN"
- note added: "VCC"
- moved on the sheet: JP1

Commit message: update
Parts:
- J1: footprint (none) -> Connectors_Samtec:SL-103-X-XX_1x03
Changed lines of the file:
@@
 LIBS:contrib
 LIBS:valves
+LIBS:touch-cache
 EELAYER 25 0
 EELAYER END
@@
 F 0 "J1" H 7230 4000 50  0000 C CNN
 F 1 "CONN_01X03" H 7380 3600 50  0000 C CNN
-F 2 "" H 7230 3800 50  0001 C CNN
+F 2 "Connectors_Samtec:SL-103-X-XX_1x03" H 7230 3800 50  0001 C CNN
 F 3 "" H 7230 3800 50  0001 C CNN
 	1    7230 3800

Commit message: update
Parts:
- 2M1: renamed from 2M; footprint (none) -> Touch_conn:res
- J1: footprint Connectors_Samtec:SL-103-X-XX_1x03 -> Touch_conn:touch_conn
- JP1: footprint (none) -> Touch_conn:touch
Changed lines of the file:
@@
 F 0 "JP1" H 6050 3129 50  0000 C CNN
 F 1 "touch" H 6060 2990 50  0000 C CNN
-F 2 "" H 6050 3050 50  0001 C CNN
+F 2 "Touch_conn:touch" H 6050 3050 50  0001 C CNN
 F 3 "" H 6050 3050 50  0001 C CNN
 	1    6050 3050
@@
 F 0 "J1" H 7230 4000 50  0000 C CNN
 F 1 "CONN_01X03" H 7380 3600 50  0000 C CNN
-F 2 "Connectors_Samtec:SL-103-X-XX_1x03" H 7230 3800 50  0001 C CNN
+F 2 "Touch_conn:touch_conn" H 7230 3800 50  0001 C CNN
 F 3 "" H 7230 3800 50  0001 C CNN
 	1    7230 3800
@@
 $EndComp
 $Comp
-L GND #PWR?
+L GND #PWR1
 U 1 1 5AFBC7A9
 P 6950 4280
-F 0 "#PWR?" H 6950 4030 50  0001 C CNN
+F 0 "#PWR1" H 6950 4030 50  0001 C CNN
 F 1 "GND" H 6950 4130 50  0000 C CNN
 F 2 "" H 6950 4280 50  0001 C CNN
@@
 $EndComp
 $Comp
-L R 2M
+L R 2M1
 U 1 1 5AFBC9A2
 P 6690 3700
-F 0 "2M" V 6770 3700 50  0000 C CNN
+F 0 "2M1" V 6770 3700 50  0000 C CNN
 F 1 "R" V 6690 3700 50  0000 C CNN
-F 2 "" V 6620 3700 50  0001 C CNN
+F 2 "Touch_conn:res" V 6620 3700 50  0001 C CNN
 F 3 "" H 6690 3700 50  0001 C CNN
 	1    6690 3700

Commit message: update
- still working
Parts:
- removed 2M1: R, Touch_conn:res, symbol R
- removed J1: CONN_01X03, Touch_conn:touch_conn, symbol CONN_01X03
- added J?: CONN_01X02, symbol CONN_01X02
Connections:
- net GND: now also J?.2 (P2)
- net at JP1.2: now also J?.1 (P1)
Other:
- note removed: "VCC"
Changed lines of the file:
@@
-$EndComp
-$Comp
-L CONN_01X03 J1
-U 1 1 5AFBC747
-P 7230 3800
-F 0 "J1" H 7230 4000 50  0000 C CNN
-F 1 "CONN_01X03" H 7380 3600 50  0000 C CNN
-F 2 "Touch_conn:touch_conn" H 7230 3800 50  0001 C CNN
-F 3 "" H 7230 3800 50  0001 C CNN
-	1    7230 3800
-	1    0    0    -1
 $EndComp
 $Comp
@@
 	1    0    0    -1
 $EndComp
-$Comp
-L R 2M1
-U 1 1 5AFBC9A2
-P 6690 3700
-F 0 "2M1" V 6770 3700 50  0000 C CNN
-F 1 "R" V 6690 3700 50  0000 C CNN
-F 2 "Touch_conn:res" V 6620 3700 50  0001 C CNN
-F 3 "" H 6690 3700 50  0001 C CNN
-	1    6690 3700
-	0    1    1    0
-$EndComp
-Text Notes 7320 3710 0    47   ~ 0
-VCC
-Text Notes 7320 3810 0    47   ~ 0
+Text Notes 7330 3830 0    47   ~ 0
 IN
 Text Notes 7320 3930 0    47   ~ 0
@@
 Wire Wire Line
 	6950 3900 6950 4280
-Wire Wire Line
-	7030 3700 6840 3700
 Wire Wire Line
 	7030 3800 6880 3800
@@
 	6410 3830 6410 3050
 Wire Wire Line
-	6410 3700 6540 3700
-Wire Wire Line
 	6410 3050 6150 3050
-Connection ~ 6410 3700
 Wire Wire Line
 	5950 3050 5670 3050
@@
 Wire Notes Line
 	6180 3180 6180 2900
+$Comp
+L CONN_01X02 J?
+U 1 1 5B018E1F
+P 7230 3850
+F 0 "J?" H 7230 4000 50  0000 C CNN
+F 1 "CONN_01X02" H 7310 3680 50  0000 C CNN
+F 2 "" H 7230 3850 50  0001 C CNN
+F 3 "" H 7230 3850 50  0001 C CNN
+	1    7230 3850
+	1    0    0    -1
+$EndComp
 $EndSCHEMATC

Commit message: update
- drawing buttons
- still to finish
Parts:
- J1: renamed from J?; footprint (none) -> Touch_conn:touch_face
- JP1: footprint Touch_conn:touch -> Touch_conn:touch_conn
Changed lines of the file:
@@
 F 0 "JP1" H 6050 3129 50  0000 C CNN
 F 1 "touch" H 6060 2990 50  0000 C CNN
-F 2 "Touch_conn:touch" H 6050 3050 50  0001 C CNN
+F 2 "Touch_conn:touch_conn" H 6050 3050 50  0001 C CNN
 F 3 "" H 6050 3050 50  0001 C CNN
 	1    6050 3050
@@
 $EndComp
 $Comp
-L GND #PWR1
+L GND #PWR01
 U 1 1 5AFBC7A9
 P 6950 4280
-F 0 "#PWR1" H 6950 4030 50  0001 C CNN
+F 0 "#PWR01" H 6950 4030 50  0001 C CNN
 F 1 "GND" H 6950 4130 50  0000 C CNN
 F 2 "" H 6950 4280 50  0001 C CNN
@@
 	6180 3180 6180 2900
 $Comp
-L CONN_01X02 J?
+L CONN_01X02 J1
 U 1 1 5B018E1F
 P 7230 3850
-F 0 "J?" H 7230 4000 50  0000 C CNN
+F 0 "J1" H 7230 4000 50  0000 C CNN
 F 1 "CONN_01X02" H 7310 3680 50  0000 C CNN
-F 2 "" H 7230 3850 50  0001 C CNN
+F 2 "Touch_conn:touch_face" H 7230 3850 50  0001 C CNN
 F 3 "" H 7230 3850 50  0001 C CNN
 	1    7230 3850

Commit message: update
- try to make a better button
Parts:
- J1: footprint Touch_conn:touch_face -> Touch_conn:touch_conn
- JP1: footprint Touch_conn:touch_conn -> Touch_conn:touch
Changed lines of the file:
@@
 LIBS:contrib
 LIBS:valves
+LIBS:my_lib
 LIBS:touch-cache
 EELAYER 25 0
@@
 F 0 "JP1" H 6050 3129 50  0000 C CNN
 F 1 "touch" H 6060 2990 50  0000 C CNN
-F 2 "Touch_conn:touch_conn" H 6050 3050 50  0001 C CNN
+F 2 "Touch_conn:touch" H 6050 3050 50  0001 C CNN
 F 3 "" H 6050 3050 50  0001 C CNN
 	1    6050 3050
@@
 F 0 "J1" H 7230 4000 50  0000 C CNN
 F 1 "CONN_01X02" H 7310 3680 50  0000 C CNN
-F 2 "Touch_conn:touch_face" H 7230 3850 50  0001 C CNN
+F 2 "Touch_conn:touch_conn" H 7230 3850 50  0001 C CNN
 F 3 "" H 7230 3850 50  0001 C CNN
 	1    7230 3850
