File: kicad/touch_button_simple/touch.sch (KiCad schematic (older format))
At the start: 2 parts, among them J1 CONN_01X02

Commit message: update
Parts:
- J1: footprint Touch_conn:touch_conn -> Touch_conn:touch_conn_cap
- JP1: footprint Touch_conn:touch -> Touch_conn:touch_zig_pro
Changed lines of the file:
@@
 F 0 "JP1" H 6050 3129 50  0000 C CNN
 F 1 "touch" H 6060 2990 50  0000 C CNN
-F 2 "Touch_conn:touch" H 6050 3050 50  0001 C CNN
+F 2 "Touch_conn:touch_zig_pro" H 6050 3050 50  0001 C CNN
 F 3 "" H 6050 3050 50  0001 C CNN
 	1    6050 3050
@@
 F 0 "J1" H 7230 4000 50  0000 C CNN
 F 1 "CONN_01X02" H 7310 3680 50  0000 C CNN
-F 2 "Touch_conn:touch_conn" H 7230 3850 50  0001 C CNN
+F 2 "Touch_conn:touch_conn_cap" H 7230 3850 50  0001 C CNN
 F 3 "" H 7230 3850 50  0001 C CNN
 	1    7230 3850
