File: kicad/touch_button_simple/touch.kicad_pcb (KiCad board)
At the start: 2 copper layers, 15 x 15 mm, 2 parts, among them J1 CONN_01X02

Commit message: update
Parts:
- JP1: footprint Touch_conn:touch_zig_pro -> touch_two_pad
Routing:
- net Net-(J1-Pad1): track 14.4 -> 18.9 mm
- net GND: track 21.9 -> 19.1 mm
Changed lines of the file:
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@@
 (kicad_pcb (version 4) (host pcbnew 4.0.6)
   (general
-    (links 35)
-    (no_connects 18)
+    (links 4)
+    (no_connects 0)
     (area 149.924999 89.924999 165.075001 105.075001)
     (thickness 1.6)
     (drawings 6)
-    (tracks 13)
+    (tracks 12)
     (zones 0)
     (modules 2)
@@
     (add_net "Net-(J1-Pad1)")
   )
+  (module touch_two_pad (layer F.Cu)
+    (at 157.48 97.536)
+    (fp_text reference JP1 (at 0 9.652) (layer F.Fab)
+      (effects (font (size 1 1) (thickness 0.15)))
+    )
+    (fp_text value touch (at 0 8.128) (layer F.Fab)
+      (effects (font (size 1 1) (thickness 0.15)))
+    )
+    (fp_line (start -7 7) (end 7 7) (layer F.SilkS) (width 0.15))
+    (fp_line (start 7 7) (end 7 -7) (layer F.SilkS) (width 0.15))
+    (fp_line (start -7 -7) (end 7 -7) (layer F.SilkS) (width 0.15))
+    (fp_line (start -7 7) (end -7 -7) (layer F.SilkS) (width 0.15))
+    (pad 2 smd oval (at 3.302 0) (size 6 13) (layers F.Cu F.Paste F.Mask)
+      (net 2 "Net-(J1-Pad1)"))
+    (pad 1 smd oval (at -3.302 0) (size 6 13) (layers F.Cu F.Paste F.Mask)
+      (net 1 GND))
+  )
   (module Touch_conn:touch_conn_cap (layer B.Cu)
     (at 157.48 97.79 90)
@@
     (pad 1 smd rect (at 2.032 4.064 90) (size 6 4) (layers B.Cu B.Paste B.Mask)
       (net 2 "Net-(J1-Pad1)"))
-  )
-  (module Touch_conn:touch_zig_pro (layer F.Cu)
-    (at 157.48 97.536)
-    (fp_text reference JP1 (at 0 9.652) (layer F.Fab)
-      (effects (font (size 1 1) (thickness 0.15)))
-    )
-    (fp_text value touch (at 0 8.128) (layer F.Fab)
-      (effects (font (size 1 1) (thickness 0.15)))
-    )
-    (fp_line (start -7 7) (end 7 7) (layer F.SilkS) (width 0.15))
-    (fp_line (start 7 7) (end 7 -7) (layer F.SilkS) (width 0.15))
-    (fp_line (start -7 -7) (end 7 -7) (layer F.SilkS) (width 0.15))
-    (fp_line (start -7 7) (end -7 -7) (layer F.SilkS) (width 0.15))
-    (pad 1 smd oval (at 2.54 2.54) (size 2 3) (layers F.Cu F.Paste F.Mask)
-      (net 1 GND))
-    (pad 2 smd oval (at -0.508 5.08) (size 2 3) (layers F.Cu F.Paste F.Mask)
-      (net 2 "Net-(J1-Pad1)"))
-    (pad 1 smd oval (at -2.794 2.54) (size 2 3) (layers F.Cu F.Paste F.Mask)
-      (net 1 GND))
-    (pad 2 smd oval (at 3.048 -3.048) (size 4 2) (layers F.Cu F.Paste F.Mask)
-      (net 2 "Net-(J1-Pad1)"))
-    (pad 1 smd oval (at -1.524 -3.048) (size 4 2) (layers F.Cu F.Paste F.Mask)
-      (net 1 GND))
-    (pad 2 smd oval (at 1.27 -0.508) (size 4 2) (layers F.Cu F.Paste F.Mask)
-      (net 2 "Net-(J1-Pad1)"))
-    (pad 2 smd oval (at -1.778 5.588) (size 4 2) (layers F.Cu F.Paste F.Mask)
-      (net 2 "Net-(J1-Pad1)"))
-    (pad 1 smd oval (at -3.302 -3.048) (size 4 2) (layers F.Cu F.Paste F.Mask)
-      (net 1 GND))
-    (pad 2 smd oval (at 4.572 -3.048) (size 3 2) (layers F.Cu F.Paste F.Mask)
-      (net 2 "Net-(J1-Pad1)"))
-    (pad 2 smd oval (at 5.334 2.032) (size 2 4) (layers F.Cu F.Paste F.Mask)
-      (net 2 "Net-(J1-Pad1)"))
-    (pad 1 smd oval (at -5.334 -0.508) (size 2 4) (layers F.Cu F.Paste F.Mask)
-      (net 1 GND))
-    (pad 1 smd oval (at 1.524 2.032) (size 4 2) (layers F.Cu F.Paste F.Mask)
-      (net 1 GND))
-    (pad 1 smd oval (at 0.254 2.032) (size 4 2) (layers F.Cu F.Paste F.Mask)
-      (net 1 GND))
-    (pad 1 smd oval (at -1.778 2.032) (size 4 2) (layers F.Cu F.Paste F.Mask)
-      (net 1 GND))
-    (pad 1 smd oval (at -3.81 2.032) (size 4 2) (layers F.Cu F.Paste F.Mask)
-      (net 1 GND))
-    (pad 1 smd oval (at -3.302 -0.508) (size 4 2) (layers F.Cu F.Paste F.Mask)
-      (net 1 GND))
-    (pad 2 smd oval (at 3.302 -0.508) (size 4 2) (layers F.Cu F.Paste F.Mask)
-      (net 2 "Net-(J1-Pad1)"))
-    (pad 2 smd oval (at 5.334 -2.032) (size 2 4) (layers F.Cu F.Paste F.Mask)
-      (net 2 "Net-(J1-Pad1)"))
-    (pad 2 smd oval (at 5.334 0) (size 2 4) (layers F.Cu F.Paste F.Mask)
-      (net 2 "Net-(J1-Pad1)"))
-    (pad 2 smd oval (at 5.334 2.286) (size 2 4) (layers F.Cu F.Paste F.Mask)
-      (net 2 "Net-(J1-Pad1)"))
-    (pad 2 smd oval (at 5.334 4.318) (size 2 4) (layers F.Cu F.Paste F.Mask)
-      (net 2 "Net-(J1-Pad1)"))
-    (pad 2 smd oval (at 2.286 5.588) (size 4 2) (layers F.Cu F.Paste F.Mask)
-      (net 2 "Net-(J1-Pad1)"))
-    (pad 2 smd oval (at 4.318 5.588) (size 4 2) (layers F.Cu F.Paste F.Mask)
-      (net 2 "Net-(J1-Pad1)"))
-    (pad 2 smd oval (at 0.254 5.588) (size 4 2) (layers F.Cu F.Paste F.Mask)
-      (net 2 "Net-(J1-Pad1)"))
-    (pad 1 smd oval (at -5.334 4.318) (size 2 4) (layers F.Cu F.Paste F.Mask)
-      (net 1 GND))
-    (pad 1 smd oval (at -5.334 2.286) (size 2 4) (layers F.Cu F.Paste F.Mask)
-      (net 1 GND))
-    (pad 1 smd oval (at -5.334 0.254) (size 2 4) (layers F.Cu F.Paste F.Mask)
-      (net 1 GND))
-    (pad 1 smd oval (at -5.334 -2.54) (size 2 4) (layers F.Cu F.Paste F.Mask)
-      (net 1 GND))
-    (pad 1 smd oval (at 1.778 -5.588) (size 4 2) (layers F.Cu F.Paste F.Mask)
-      (net 1 GND))
-    (pad 1 smd oval (at -0.254 -5.588) (size 4 2) (layers F.Cu F.Paste F.Mask)
-      (net 1 GND))
-    (pad 1 smd oval (at -2.286 -5.588) (size 4 2) (layers F.Cu F.Paste F.Mask)
-      (net 1 GND))
-    (pad 1 smd oval (at -4.318 -5.588) (size 4 2) (layers F.Cu F.Paste F.Mask)
-      (net 1 GND))
-    (pad 1 smd oval (at -5.334 -4.318) (size 2 4) (layers F.Cu F.Paste F.Mask)
-      (net 1 GND))
   )
   (gr_line (start 150 90) (end 165 90) (angle 90) (layer Edge.Cuts) (width 0.15))
@@
   (gr_line (start 165 90) (end 165 105) (angle 90) (layer Edge.Cuts) (width 0.15))
   (gr_line (start 150 90) (end 150 105) (angle 90) (layer Edge.Cuts) (width 0.15))
-  (segment (start 153.416 95.758) (end 153.416 101.854) (width 0.25) (layer B.Cu) (net 1) (status C00000))
-  (segment (start 161.798 91.948) (end 159.258 91.948) (width 0.25) (layer F.Cu) (net 1))
-  (segment (start 162.56 91.186) (end 161.798 91.948) (width 0.25) (layer F.Cu) (net 1))
-  (via (at 162.56 91.186) (size 0.6) (drill 0.4) (layers F.Cu B.Cu) (net 1))
-  (segment (start 155.956 91.186) (end 162.56 91.186) (width 0.25) (layer B.Cu) (net 1))
-  (segment (start 153.416 93.726) (end 155.956 91.186) (width 0.25) (layer B.Cu) (net 1))
-  (segment (start 153.416 95.758) (end 153.416 93.726) (width 0.25) (layer B.Cu) (net 1))
-  (segment (start 161.544 95.758) (end 161.544 101.854) (width 0.25) (layer B.Cu) (net 2) (status C00000))
-  (segment (start 161.544 95.758) (end 161.544 93.726) (width 0.25) (layer B.Cu) (net 2))
-  (segment (start 161.544 93.726) (end 163.322 91.948) (width 0.25) (layer B.Cu) (net 2))
-  (via (at 163.322 91.948) (size 0.6) (drill 0.4) (layers F.Cu B.Cu) (net 2))
-  (segment (start 163.322 91.948) (end 162.814 92.456) (width 0.25) (layer F.Cu) (net 2))
-  (segment (start 162.814 92.456) (end 162.814 95.504) (width 0.25) (layer F.Cu) (net 2))
+  (segment (start 153.416 95.758) (end 153.416 93.2815) (width 0.25) (layer B.Cu) (net 1))
+  (segment (start 153.416 93.2815) (end 151.3205 91.186) (width 0.25) (layer B.Cu) (net 1))
+  (segment (start 151.3205 91.186) (end 154.178 94.0435) (width 0.25) (layer F.Cu) (net 1))
+  (via (at 151.3205 91.186) (size 0.6) (drill 0.4) (layers F.Cu B.Cu) (net 1))
+  (segment (start 154.178 94.0435) (end 154.178 97.536) (width 0.25) (layer F.Cu) (net 1))
+  (segment (start 153.416 95.758) (end 153.416 101.854) (width 0.25) (layer B.Cu) (net 1))
+  (segment (start 161.544 95.758) (end 161.544 93.5355) (width 0.25) (layer B.Cu) (net 2) (status C00000))
+  (segment (start 161.544 93.5355) (end 163.7665 91.313) (width 0.25) (layer B.Cu) (net 2) (status 400000))
+  (segment (start 163.7665 91.313) (end 160.782 94.2975) (width 0.25) (layer F.Cu) (net 2) (status 800000))
+  (via (at 163.7665 91.313) (size 0.6) (drill 0.4) (layers F.Cu B.Cu) (net 2))
+  (segment (start 160.782 94.2975) (end 160.782 97.536) (width 0.25) (layer F.Cu) (net 2) (status C00000))
+  (segment (start 161.544 95.758) (end 161.544 101.854) (width 0.25) (layer B.Cu) (net 2))
 )
